Commit message: feat: adjust camera joint orientation for improved ground visibility

File: src/alphabot2_gazebo/urdf/alphabot2.urdf (robot description, URDF)
Before this commit: robot alphabot2, 7 links, 6 joints
Joints:
- joint camera_joint: origin xyz=0.040 0 0.060 rpy=0 0.10 0 -> xyz=0.040 0 0.060 rpy=0 0.7854 0
